File: OSLUV.kicad_sch (KiCad schematic)
At the start: 7 parts, among them J7 B5P-VH

Commit message: Rev. 1.0.0 production data
Parts:
- removed H5: MountingHole_Pad, Hansmann:Mounting_M3_NPTH_Vias, symbol Mechanical:MountingHole_Pad
- renumbered J7 to J6
Changed lines of the file:
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@@
 	(paper "A4")
-	(junction
-		(at 118.11 119.38)
-		(diameter 0)
-		(color 0 0 0 0)
-	)
 	(junction
 		(at 106.68 119.38)
@@
 	(wire
 		(pts
-			(xy 118.11 119.38) (xy 201.93 119.38)
+			(xy 106.68 119.38) (xy 201.93 119.38)
 		)
 		(stroke
@@
 		(pts
 			(xy 229.87 93.98) (xy 229.87 96.52)
-		)
-		(stroke
-			(width 0)
-			(type default)
-		)
-	)
-	(wire
-		(pts
-			(xy 106.68 119.38) (xy 118.11 119.38)
 		)
 		(stroke
@@
 	)
 	(symbol
-		(lib_id "Mechanical:MountingHole_Pad")
-		(at 118.11 121.92 180)
-		(unit 1)
-		(exclude_from_sim no)
-		(in_bom no)
-		(on_board yes)
-		(dnp no)
-		(property "Reference" "H5"
-			(at 117.094 127 0)
-			(effects
-				(font
-					(size 1.27 1.27)
-				)
-				(justify right)
-			)
-		)
-		(property "Value" "MountingHole_Pad"
-			(at 110.744 127 0)
-			(effects
-				(font
-					(size 1.27 1.27)
-				)
-				(justify right)
-				(hide yes)
-			)
-		)
-		(property "Footprint" "Hansmann:Mounting_M3_NPTH_Vias"
-			(at 118.11 121.92 0)
-			(effects
-				(font
-					(size 1.27 1.27)
-				)
-				(hide yes)
-			)
-		)
-		(property "Datasheet" ""
-			(at 118.11 121.92 0)
-			(effects
-				(font
-					(size 1.27 1.27)
-				)
-				(hide yes)
-			)
-		)
-		(property "Description" "Mounting Hole with connection"
-			(at 118.11 121.92 0)
-			(effects
-				(font
-					(size 1.27 1.27)
-				)
-				(hide yes)
-			)
-		)
-		(pin "1"
-		)
-		(instances
-			(project "OSLUV"
-				(path "/c6e900e0-9399-44f0-8089-9dd7b8ffe54c"
-					(reference "H5")
-					(unit 1)
-				)
-			)
-		)
-	)
-	(symbol
 		(lib_id "Hansmann:B2P5-VH")
 		(at 238.76 96.52 0)
@@
 		(dnp no)
 		(fields_autoplaced yes)
-		(property "Reference" "J7"
+		(property "Reference" "J6"
 			(at 247.65 78.74 0)
 			(effects
@@
 			(project ""
 				(path "/c6e900e0-9399-44f0-8089-9dd7b8ffe54c"
-					(reference "J7")
+					(reference "J6")
 					(unit 1)
 				)
