File: OSLUV.kicad_sch (KiCad schematic)
At the start: 3 parts, among them J6 B5P-VH

Commit message: part correction
Other:
- moved on the sheet: H3, H4, J6
Changed lines of the file:
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@@
 	(paper "A4")
 	(junction
-		(at 193.04 118.11)
+		(at 125.73 123.19)
 		(diameter 0)
 		(color 0 0 0 0)
@@
 	(wire
 		(pts
-			(xy 182.88 118.11) (xy 193.04 118.11)
+			(xy 115.57 123.19) (xy 125.73 123.19)
 		)
 		(stroke
@@
 	(wire
 		(pts
-			(xy 201.93 118.11) (xy 201.93 113.03)
+			(xy 134.62 123.19) (xy 134.62 118.11)
 		)
 		(stroke
@@
 	(wire
 		(pts
-			(xy 229.87 96.52) (xy 238.76 96.52)
+			(xy 156.21 91.44) (xy 171.45 91.44)
 		)
 		(stroke
@@
 	(wire
 		(pts
-			(xy 223.52 86.36) (xy 238.76 86.36)
+			(xy 125.73 123.19) (xy 134.62 123.19)
 		)
 		(stroke
@@
 	(wire
 		(pts
-			(xy 193.04 118.11) (xy 201.93 118.11)
+			(xy 156.21 101.6) (xy 171.45 101.6)
 		)
 		(stroke
@@
 		)
 	)
-	(wire
-		(pts
-			(xy 223.52 93.98) (xy 229.87 93.98)
-		)
-		(stroke
-			(width 0)
-			(type default)
-		)
-	)
-	(wire
-		(pts
-			(xy 229.87 93.98) (xy 229.87 96.52)
-		)
-		(stroke
-			(width 0)
-			(type default)
-		)
-	)
 	(netclass_flag ""
 		(length 2.54)
 		(shape round)
-		(at 201.93 118.11 180)
+		(at 134.62 123.19 180)
 		(fields_autoplaced yes)
 		(effects
@@
 		)
 		(property "Netclass" "MAINS_preFuse"
-			(at 202.5396 120.65 0)
+			(at 135.2296 125.73 0)
 			(effects
 				(font
@@
 		)
 		(property "Component Class" ""
-			(at -39.37 0 0)
+			(at -106.68 5.08 0)
 			(effects
 				(font
@@
 	(symbol
 		(lib_id "Mechanical:MountingHole_Pad")
-		(at 193.04 120.65 180)
+		(at 125.73 125.73 180)
 		(unit 1)
 		(exclude_from_sim no)
@@
 		(dnp no)
 		(property "Reference" "H4"
-			(at 192.024 125.73 0)
+			(at 124.714 130.81 0)
 			(effects
 				(font
@@
 		)
 		(property "Value" "MountingHole_Pad"
-			(at 185.674 125.73 0)
+			(at 118.364 130.81 0)
 			(effects
 				(font
@@
 		)
 		(property "Footprint" "Hansmann:Mounting_M3_NPTH_Vias"
-			(at 193.04 120.65 0)
+			(at 125.73 125.73 0)
 			(effects
 				(font
@@
 		)
 		(property "Datasheet" ""
-			(at 193.04 120.65 0)
+			(at 125.73 125.73 0)
 			(effects
 				(font
@@
 		)
 		(property "Description" "Mounting Hole with connection"
-			(at 193.04 120.65 0)
+			(at 125.73 125.73 0)
 			(effects
 				(font
@@
 		)
 		(property "Arrow Part Number" ""
-			(at 193.04 120.65 0)
+			(at 125.73 125.73 0)
 			(effects
 				(font
@@
 		)
 		(property "Arrow Price/Stock" ""
-			(at 193.04 120.65 0)
+			(at 125.73 125.73 0)
 			(effects
 				(font
@@
 		)
 		(property "Field10" ""
-			(at 193.04 120.65 0)
+			(at 125.73 125.73 0)
 			(effects
 				(font
@@
 		)
 		(property "L (mH)" ""
-			(at 193.04 120.65 0)
+			(at 125.73 125.73 0)
 			(effects
 				(font
@@
 		)
 		(property "Material" ""
-			(at 193.04 120.65 0)
+			(at 125.73 125.73 0)
 			(effects
 				(font
@@
 		)
 		(property "RDC max. (mΩ)" ""
-			(at 193.04 120.65 0)
+			(at 125.73 125.73 0)
 			(effects
 				(font
@@
 		)
 		(property "VT (V (AC))" ""
-			(at 193.04 120.65 0)
+			(at 125.73 125.73 0)
 			(effects
 				(font
@@
 	(symbol
 		(lib_id "Hansmann:B2P5-VH")
-		(at 238.76 96.52 0)
+		(at 171.45 101.6 0)
 		(mirror x)
 		(unit 1)
@@
 		(fields_autoplaced yes)
 		(property "Reference" "J6"
-			(at 247.65 78.74 0)
+			(at 180.34 83.82 0)
 			(effects
 				(font
@@
 		)
 		(property "Value" "B5P-VH"
-			(at 247.65 81.28 0)
+			(at 180.34 86.36 0)
 			(effects
 				(font
@@
 		)
 		(property "Footprint" "Hansmann:CONN_B2P5-VH_JST"
-			(at 238.76 96.52 0)
+			(at 171.45 101.6 0)
 			(effects
 				(font
@@
 		)
 		(property "Datasheet" "B5P-VH"
-			(at 238.76 96.52 0)
+			(at 171.45 101.6 0)
 			(effects
 				(font
@@
 		)
 		(property "Description" ""
-			(at 238.76 96.52 0)
+			(at 171.45 101.6 0)
 			(effects
 				(font
@@
 		)
 		(property "Arrow Part Number" ""
-			(at 238.76 96.52 0)
+			(at 171.45 101.6 0)
 			(effects
 				(font
@@
 		)
 		(property "Arrow Price/Stock" ""
-			(at 238.76 96.52 0)
+			(at 171.45 101.6 0)
 			(effects
 				(font
@@
 		)
 		(property "Field10" ""
-			(at 238.76 96.52 0)
+			(at 171.45 101.6 0)
 			(effects
 				(font
@@
 		)
 		(property "L (mH)" ""
-			(at 238.76 96.52 0)
+			(at 171.45 101.6 0)
 			(effects
 				(font
@@
 		)
 		(property "Material" ""
-			(at 238.76 96.52 0)
+			(at 171.45 101.6 0)
 			(effects
 				(font
@@
 		)
 		(property "RDC max. (mΩ)" ""
-			(at 238.76 96.52 0)
+			(at 171.45 101.6 0)
 			(effects
 				(font
@@
 		)
 		(property "VT (V (AC))" ""
-			(at 238.76 96.52 0)
+			(at 171.45 101.6 0)
 			(effects
 				(font
@@
 	(symbol
 		(lib_id "Mechanical:MountingHole_Pad")
-		(at 182.88 120.65 180)
+		(at 115.57 125.73 180)
 		(unit 1)
 		(exclude_from_sim no)
@@
 		(dnp no)
 		(property "Reference" "H3"
-			(at 181.864 125.73 0)
+			(at 114.554 130.81 0)
 			(effects
 				(font
@@
 		)
 		(property "Value" "MountingHole_Pad"
-			(at 175.514 125.73 0)
+			(at 108.204 130.81 0)
 			(effects
 				(font
@@
 		)
 		(property "Footprint" "Hansmann:Mounting_M3_NPTH_Vias"
-			(at 182.88 120.65 0)
+			(at 115.57 125.73 0)
 			(effects
 				(font
@@
 		)
 		(property "Datasheet" ""
-			(at 182.88 120.65 0)
+			(at 115.57 125.73 0)
 			(effects
 				(font
@@
 		)
 		(property "Description" "Mounting Hole with connection"
-			(at 182.88 120.65 0)
+			(at 115.57 125.73 0)
 			(effects
 				(font
@@
 		)
 		(property "Arrow Part Number" ""
-			(at 182.88 120.65 0)
+			(at 115.57 125.73 0)
 			(effects
 				(font
@@
 		)
 		(property "Arrow Price/Stock" ""
-			(at 182.88 120.65 0)
+			(at 115.57 125.73 0)
 			(effects
 				(font
@@
 		)
 		(property "Field10" ""
-			(at 182.88 120.65 0)
+			(at 115.57 125.73 0)
 			(effects
 				(font
@@
 		)
 		(property "L (mH)" ""
-			(at 182.88 120.65 0)
+			(at 115.57 125.73 0)
 			(effects
 				(font
@@
 		)
 		(property "Material" ""
-			(at 182.88 120.65 0)
+			(at 115.57 125.73 0)
 			(effects
 				(font
@@
 		)
 		(property "RDC max. (mΩ)" ""
-			(at 182.88 120.65 0)
+			(at 115.57 125.73 0)
 			(effects
 				(font
@@
 		)
 		(property "VT (V (AC))" ""
-			(at 182.88 120.65 0)
+			(at 115.57 125.73 0)
 			(effects
 				(font
@@
 	)
 	(sheet
-		(at 165.1 67.31)
+		(at 97.79 72.39)
 		(size 58.42 45.72)
 		(exclude_from_sim no)
@@
 		)
 		(property "Sheetname" "excimerDriver"
-			(at 165.1 66.5984 0)
+			(at 97.79 71.6784 0)
 			(effects
 				(font
@@
 		)
 		(property "Sheetfile" "excimerDriver.kicad_sch"
-			(at 165.1 113.6146 0)
+			(at 97.79 118.6946 0)
 			(effects
 				(font
@@
 		)
 		(pin "EARTH" passive
-			(at 201.93 113.03 270)
+			(at 134.62 118.11 270)
 			(effects
 				(font
@@
 		)
 		(pin "Lamp_GND" passive
-			(at 223.52 93.98 0)
+			(at 156.21 101.6 0)
 			(effects
 				(font
@@
 		)
 		(pin "Lamp_HV" passive
-			(at 223.52 86.36 0)
-			(effects
-				(font
+			(at 156.21 91.44 0)
+			(effects
+				(font
