File: OSLUV.kicad_pcb (KiCad board)
At the start: 4 copper layers, 110 x 40 mm, 160 parts, among them IC1 OPA2356AIDGKR, IC2 LM2901, IC3 STM32G071KBT6, IC4 INA210, IC5 AP63300WU-7, IC6 AP63300WU-7, IC7 LP2985-33DBVR, IC8 1ED44175N01BXTSA1, J1 B04B-XASK-1_LF__SN_, J2 B08B-XASK-1-A_LF__SN_, J3 TC2030, J4 BM02B-SRSS-TB_LF__SN_, J5 B4B-PH-K-S_LF__SN_, J6 B5P-VH, M1 K 274 MI 247 V, M2 KU-CG20, T101 IMZC120R078M2H, T2 DCX114EU-7-F, T3 BC817-40, T4 DCX114EU-7-F, T5 DCX114EU-7-F

Commit message: part correction
Parts:
- C16, C17, C43, C45, C47, C5, C56: value 10µ X7R 1210 -> 10µ X7R 1210 50V
- C30, C31, C36, C37, C39: value 10u X7R 1210 -> 10µ X7R 1210 50V
- C49: value 10p 1% 600V 1206 -> 10p 1% 500V 1206
- IC4: value INA210 -> INA210AIDCKJ
- R67, R68: value 1Meg 0.1% 500V 1206 -> 1Meg 1% 500V 1206
