File: excimerDriver.kicad_sch (KiCad schematic)
At the start: 60 parts, among them IC3 STM32G071KBT6, IC4 INA210, J1 B04B-XASK-1_LF__SN_, J2 B08B-XASK-1-A_LF__SN_, J3 TC2030, J4 BM02B-SRSS-TB_LF__SN_, J5 B4B-PH-K-S_LF__SN_, T2 DCX114EU-7-F, T3 BC817-40

Commit message: part correction
Parts:
- C16, C17, C5: value 10µ X7R 1210 -> 10µ X7R 1210 50V
- D13: Manufacturer  (none) -> Diodes Incorporated; Manufacturer Part Number (none) -> D5V0P4UR6SO-7; Manufacturer_Name Diodes Incorporated -> (none); Manufacturer_Part_Number D5V0P4UR6SO-7 -> (none)
- D14: Manufacturer (none) -> Diodes Incorporated; Manufacturer Part Number (none) -> D5V0P4UR6SO-7; Manufacturer_Name Diodes Incorporated -> (none); Manufacturer_Part_Number D5V0P4UR6SO-7 -> (none)
- IC3: Manufacturer (none) -> STMicroelectronics; Manufacturer Part Number (none) -> STM32G071KBT6; Manufacturer_Name STMicroelectronics -> (none); Manufacturer_Part_Number STM32G071KBT6 -> (none)
- IC4: value INA210 -> INA210AIDCKJ; Manufacturer (none) -> Texas Instruments; Manufacturer Part Number (none) -> INA210AIDCKJ
- J1: Manufacturer  (none) -> JST (JAPAN SOLDERLESS TERMINALS); Manufacturer Part Number (none) -> B04B-XASK-1(LF)(SN); Manufacturer_Name JST (JAPAN SOLDERLESS TERMINALS) -> (none); Manufacturer_Part_Number B04B-XASK-1(LF)(SN) -> (none)
- J2: Manufacturer (none) -> JST (JAPAN SOLDERLESS TERMINALS); Manufacturer Part Number (none) -> B08B-XASK-1-A(LF)(SN); Manufacturer_Name JST (JAPAN SOLDERLESS TERMINALS) -> (none); Manufacturer_Part_Number B08B-XASK-1-A(LF)(SN) -> (none)
- J4: Manufacturer  (none) -> JST (JAPAN SOLDERLESS TERMINALS); Manufacturer Part Number (none) -> BM02B-SRSS-TB(LF)(SN); Manufacturer_Name JST (JAPAN SOLDERLESS TERMINALS) -> (none); Manufacturer_Part_Number BM02B-SRSS-TB(LF)(SN) -> (none)
- J5: Manufacturer  (none) -> JST (JAPAN SOLDERLESS TERMINALS); Manufacturer Part Number (none) -> B4B-PH-K-S(LF)(SN); Manufacturer_Name JST (JAPAN SOLDERLESS TERMINALS) -> (none); Manufacturer_Part_Number B4B-PH-K-S(LF)(SN) -> (none)
- T2: Manufacturer (none) -> Diodes Incorporated; Manufacturer Part Number (none) -> DCX114EU-7-F; Manufacturer_Name Diodes Incorporated -> (none); Manufacturer_Part_Number DCX114EU-7-F -> (none)
Changed lines of the file:
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@@
 	(wire
 		(pts
+			(xy 88.9 132.08) (xy 86.36 132.08)
+		)
+		(stroke
+			(width 0)
+			(type default)
+		)
+	)
+	(wire
+		(pts
 			(xy 82.55 33.02) (xy 82.55 38.1)
 		)
@@
 	(wire
 		(pts
-			(xy 86.36 132.08) (xy 88.9 132.08)
-		)
-		(stroke
-			(width 0)
-			(type default)
-		)
-	)
-	(wire
-		(pts
 			(xy 114.3 161.29) (xy 114.3 160.02)
 		)
@@
 	)
 	(image
-		(at 67.31 243.84)
+		(at 151.13 177.8)
 		(scale 0.374311)
 		(data "iVBORw0KGgoAAAANSUhEUgAAA7EAAAJ2CAIAAAAG25K2AAAAA3NCSVQICAjb4U/gAAAACXBIWXMA"
@@
 	)
 	(label "LED1"
-		(at 86.36 132.08 180)
+		(at 88.9 132.08 180)
 		(effects
 			(font
@@
 			)
 		)
-		(property "Manufacturer_Name" "STMicroelectronics"
+		(property "Manufacturer" "STMicroelectronics"
 			(at 135.89 806.68 0)
 			(effects
@@
 			)
 		)
-		(property "Manufacturer_Part_Number" "STM32G071KBT6"
+		(property "Manufacturer Part Number" "STM32G071KBT6"
 			(at 135.89 906.68 0)
 			(effects
@@
 			)
 		)
-		(property "Manufacturer_Name" "JST (JAPAN SOLDERLESS TERMINALS)"
+		(property "Manufacturer" "JST (JAPAN SOLDERLESS TERMINALS)"
 			(at 12.7 -552.68 0)
 			(effects
@@
 			)
 		)
-		(property "Manufacturer_Part_Number" "B08B-XASK-1-A(LF)(SN)"
+		(property "Manufacturer Part Number" "B08B-XASK-1-A(LF)(SN)"
 			(at 12.7 -652.68 0)
 			(effects
@@
 			)
 		)
-		(property "Value" "10µ X7R 1210"
+		(property "Value" "10µ X7R 1210 50V"
 			(at 89.916 31.75 0)
 			(effects
@@
 			)
 		)
-		(property "Value" "10µ X7R 1210"
+		(property "Value" "10µ X7R 1210 50V"
 			(at 81.026 22.606 0)
 			(effects
@@
 			)
 		)
-		(property "Manufacturer_Name" "Diodes Incorporated"
+		(property "Manufacturer" "Diodes Incorporated"
 			(at 52.07 867.64 0)
 			(effects
@@
 			)
 		)
-		(property "Manufacturer_Part_Number" "DCX114EU-7-F"
+		(property "Manufacturer Part Number" "DCX114EU-7-F"
 			(at 52.07 967.64 0)
 			(effects
@@
 			)
 		)
-		(property "Manufacturer_Name" "JST (JAPAN SOLDERLESS TERMINALS)"
+		(property "Manufacturer " "JST (JAPAN SOLDERLESS TERMINALS)"
 			(at 252.73 156.21 0)
 			(effects
@@
 			)
 		)
-		(property "Manufacturer_Part_Number" "B4B-PH-K-S(LF)(SN)"
+		(property "Manufacturer Part Number" "B4B-PH-K-S(LF)(SN)"
 			(at 252.73 158.75 0)
 			(effects
@@
 			)
 		)
-		(property "Manufacturer_Name" "Diodes Incorporated"
+		(property "Manufacturer " "Diodes Incorporated"
 			(at 58.42 -625.07 0)
 			(effects
@@
 			)
 		)
-		(property "Manufacturer_Part_Number" "D5V0P4UR6SO-7"
+		(property "Manufacturer Part Number" "D5V0P4UR6SO-7"
 			(at 58.42 -725.07 0)
 			(effects
@@
 			)
 		)
-		(property "Manufacturer_Name" "JST (JAPAN SOLDERLESS TERMINALS)"
+		(property "Manufacturer " "JST (JAPAN SOLDERLESS TERMINALS)"
 			(at 43.18 722.86 0)
 			(effects
@@
 			)
 		)
-		(property "Manufacturer_Part_Number" "B04B-XASK-1(LF)(SN)"
+		(property "Manufacturer Part Number" "B04B-XASK-1(LF)(SN)"
 			(at 43.18 822.86 0)
 			(effects
@@
 			)
 		)
-		(property "Manufacturer_Name" "JST (JAPAN SOLDERLESS TERMINALS)"
+		(property "Manufacturer " "JST (JAPAN SOLDERLESS TERMINALS)"
 			(at 255.27 809.22 0)
 			(effects
@@
 			)
 		)
-		(property "Manufacturer_Part_Number" "BM02B-SRSS-TB(LF)(SN)"
+		(property "Manufacturer Part Number" "BM02B-SRSS-TB(LF)(SN)"
 			(at 255.27 909.22 0)
 			(effects
@@
 			)
 		)
-		(property "Manufacturer_Name" "Diodes Incorporated"
+		(property "Manufacturer" "Diodes Incorporated"
 			(at 214.63 821.92 0)
 			(effects
@@
 			)
 		)
-		(property "Manufacturer_Part_Number" "D5V0P4UR6SO-7"
+		(property "Manufacturer Part Number" "D5V0P4UR6SO-7"
 			(at 214.63 921.92 0)
 			(effects
@@
 			)
 		)
-		(property "Value" "INA210"
+		(property "Value" "INA210AIDCKJ"
 			(at 167.64 89.4649 0)
 			(effects
@@
 			)
 		)
+		(property "Manufacturer" "Texas Instruments"
+			(at 139.7 92.71 0)
+			(effects
+				(font
+					(size 1.27 1.27)
+				)
+				(hide yes)
+			)
+		)
+		(property "Manufacturer Part Number" "INA210AIDCKJ"
+			(at 139.7 92.71 0)
+			(effects
+				(font
+					(size 1.27 1.27)
+				)
+				(hide yes)
+			)
+		)
 		(pin "2"
 		)
@@
 			)
 		)
-		(property "Value" "10µ X7R 1210"
+		(property "Value" "10µ X7R 1210 50V"
 			(at 83.566 31.75 0)
 			(effects
