File: lampDriver.kicad_sch (KiCad schematic)
At the start: 74 parts, among them IC1 OPA2356AIDGKR, IC2 LM2901, IC8 1ED44175N01BXTSA1, M1 K 274 MI 247 V, M2 KU-CG20, T101 IMZC120R078M2H, T4 DCX114EU-7-F, T5 DCX114EU-7-F

Commit message: part correction
Parts:
- C43, C45, C47, C56: value 10µ X7R 1210 -> 10µ X7R 1210 50V
- C49, C50: value 10p 1% 600V 1206 -> 10p 1% 500V 1206; Manufacturer (none) -> KEMET; Manufacturer Part Number (none) -> C1206C100FCGACTU
- IC1: Manufacturer (none) -> Texas Instruments; Manufacturer Part Number (none) -> OPA2356AIDGKR
- IC2: Manufacturer (none) -> Texas Instruments; Manufacturer Part Number (none) -> LM2901BIPWR
- IC8: Manufacturer (none) -> Infineon; Manufacturer Part Number (none) -> 1ED44175N01BXTSA1; Manufacturer_Name Infineon -> (none); Manufacturer_Part_Number 1ED44175N01BXTSA1 -> (none)
- R67, R68: value 1Meg 0.1% 500V 1206 -> 1Meg 1% 500V 1206; Manufacturer (none) -> ROHM; Manufacturer Part Number (none) -> KTR18EZPF1004
- R70, R71: Manufacturer (none) -> Vishay; Manufacturer Part Number (none) -> MMA02040C1800FB300
- T101: Manufacturer (none) -> Infineon; Manufacturer Part Number (none) -> IMZC120R078M2H
- T4, T5: Manufacturer (none) -> Diodes Incorporated; Manufacturer Part Number (none) -> DCX114EU-7-F; Manufacturer_Name Diodes Incorporated -> (none); Manufacturer_Part_Number DCX114EU-7-F -> (none)
- TH1: Article B59721A0070A062 -> (none); Manufacturer (none) -> TDK; Manufacturer Part Number (none) -> B59721A0080A062
